File: flasher/flasher.sch (EAGLE design)
At the start: 48 parts, among them IC1 ULN2004A_BIG_SMD, Q1 IRF4905, Q2 IRF4905

Commit message: Change resistors value
Parts:
- R1, R4: value 100k -> 33k
- R12, R13, R14, R15: value 18k -> 4k7
- R16: value 18k -> 0R
- R2, R5: value 18k -> 5k6
- R3, R6: value 33k -> 3k3
