File: flasher/v1.1/flasher.sch (EAGLE design)
At the start: 51 parts, among them IC1 ULN2004A_BIG_SMD, IC2 7805, Q1 IRF4905, Q2 IRF4905, Q3 MMBF170, Q4 MMBF170, Q5 MMBF170, Q6 MMBF170

Commit message: Flasher v1.2: add reverse protection diode and capacitors to stabilizer, add some missing parts value, minor cosmetics changes
Parts:
- removed C2: 100n, rcl_upravena:C-EUC0805
- removed C3: 330n, rcl_upravena:C-EUC0805
- removed D3: (no value), diode:DIODE-SOD123
- C1: value 330u/16V -> (none)
- IC2: value 7805 -> (none)
- Q3, Q4, Q5, Q6: value MMBF170 -> (none)
Connections:
- net +5V: no longer C3.1, D3.A
- net GND: no longer C2.2, C3.2
- net VCC: no longer C2.1, D3.C
Other:
- note added: "v1.1"
- note removed: "v1.2"
Changed lines of the file:
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@@
 <part name="+3V1" library="supply1" deviceset="+3V3" device=""/>
 <part name="GND2" library="supply1" deviceset="GND" device=""/>
-<part name="C1" library="rcl_upravena" deviceset="CPOL-EU" device="E5-10.5" value="330u/16V"/>
+<part name="C1" library="rcl_upravena" deviceset="CPOL-EU" device="E5-10.5"/>
 <part name="GND3" library="supply1" deviceset="GND" device=""/>
 <part name="D1" library="diode" deviceset="DIODE" device="-SOD123"/>
@@
 <part name="U$5" library="piezo" deviceset="PIEZO" device=""/>
 <part name="JP1" library="pinhead_smd" deviceset="PINH2X04" device=""/>
-<part name="Q3" library="transistors" deviceset="N-MOSFET" device="-SOT23-DIST" value="MMBF170"/>
-<part name="Q4" library="transistors" deviceset="N-MOSFET" device="-SOT23-DIST" value="MMBF170"/>
+<part name="Q3" library="transistors" deviceset="N-MOSFET" device="-SOT23-DIST"/>
+<part name="Q4" library="transistors" deviceset="N-MOSFET" device="-SOT23-DIST"/>
 <part name="R12" library="rcl_upravena" deviceset="R-EU_" device="R0805S" value="4k7"/>
 <part name="R13" library="rcl_upravena" deviceset="R-EU_" device="R0805S" value="4k7"/>
 <part name="P+8" library="supply1" deviceset="+5V" device=""/>
 <part name="GND9" library="supply1" deviceset="GND" device=""/>
-<part name="Q5" library="transistors" deviceset="N-MOSFET" device="-SOT23-DIST" value="MMBF170"/>
-<part name="Q6" library="transistors" deviceset="N-MOSFET" device="-SOT23-DIST" value="MMBF170"/>
+<part name="Q5" library="transistors" deviceset="N-MOSFET" device="-SOT23-DIST"/>
+<part name="Q6" library="transistors" deviceset="N-MOSFET" device="-SOT23-DIST"/>
 <part name="R14" library="rcl_upravena" deviceset="R-EU_" device="R0805S" value="4k7"/>
 <part name="R15" library="rcl_upravena" deviceset="R-EU_" device="R0805S" value="4k7"/>
@@
 <part name="GND10" library="supply1" deviceset="GND" device=""/>
 <part name="GND11" library="supply1" deviceset="GND" device=""/>
+<part name="GND12" library="supply1" deviceset="GND" device=""/>
 <part name="R16" library="rcl_upravena" deviceset="R-EU_" device="R0805S" value="0R"/>
 <part name="NC7" library="NC" deviceset="NC" device=""/>
@@
 <part name="P+3" library="supply1" deviceset="VCC" device=""/>
 <part name="P+4" library="supply1" deviceset="VCC" device=""/>
-<part name="IC2" library="v-reg" deviceset="78XXS" device="" value="7805"/>
+<part name="IC2" library="v-reg" deviceset="78XXS" device=""/>
 <part name="P+11" library="supply1" deviceset="VCC" device=""/>
 <part name="P+12" library="supply1" deviceset="+5V" device=""/>
@@
 <part name="JP2" library="pinhead" deviceset="PINHD-1X4" device="/90"/>
 <part name="JP3" library="pinhead" deviceset="PINHD-1X5" device=""/>
-<part name="D3" library="diode" deviceset="DIODE" device="-SOD123"/>
-<part name="C2" library="rcl_upravena" deviceset="C-EU" device="C0805" value="100n"/>
-<part name="C3" library="rcl_upravena" deviceset="C-EU" device="C0805" value="330n"/>
 </parts>
 <sheets>
 <sheet>
 <plain>
-<text x="171.196" y="5.08" size="2.54" layer="94" font="vector">v1.2</text>
+<text x="171.196" y="5.08" size="2.54" layer="94" font="vector">v1.1</text>
 <text x="140.97" y="20.32" size="2.54" layer="94" font="vector">Jakub Streit</text>
 </plain>
@@
 <instance part="JP1" gate="B4" x="162.56" y="241.3" rot="MR0"/>
 <instance part="Q3" gate="G$1" x="93.98" y="238.76" smashed="yes" rot="MR90">
-<attribute name="VALUE" x="95.25" y="246.38" size="1.778" layer="96" rot="MR180"/>
+<attribute name="VALUE" x="93.98" y="227.33" size="1.778" layer="96" rot="MR90"/>
 <attribute name="NAME" x="90.17" y="246.38" size="1.778" layer="95" rot="MR180"/>
 </instance>
 <instance part="Q4" gate="G$1" x="101.6" y="233.68" smashed="yes" rot="MR90">
-<attribute name="VALUE" x="105.41" y="231.14" size="1.778" layer="96" rot="MR180"/>
+<attribute name="VALUE" x="101.6" y="222.25" size="1.778" layer="96" rot="MR90"/>
 <attribute name="NAME" x="100.33" y="231.14" size="1.778" layer="95" rot="MR180"/>
 </instance>
@@
 <instance part="GND9" gate="1" x="142.24" y="228.6"/>
 <instance part="Q5" gate="G$1" x="99.06" y="200.66" smashed="yes" rot="MR90">
-<attribute name="VALUE" x="100.33" y="208.28" size="1.778" layer="96" rot="MR180"/>
+<attribute name="VALUE" x="99.06" y="189.23" size="1.778" layer="96" rot="MR90"/>
 <attribute name="NAME" x="95.25" y="208.28" size="1.778" layer="95" rot="MR180"/>
 </instance>
 <instance part="Q6" gate="G$1" x="101.6" y="195.58" smashed="yes" rot="MR90">
-<attribute name="VALUE" x="105.41" y="193.04" size="1.778" layer="96" rot="MR180"/>
+<attribute name="VALUE" x="101.6" y="184.15" size="1.778" layer="96" rot="MR90"/>
 <attribute name="NAME" x="100.33" y="193.04" size="1.778" layer="95" rot="MR180"/>
 </instance>
@@
 <instance part="GND10" gate="1" x="142.24" y="190.5"/>
 <instance part="GND11" gate="1" x="157.48" y="228.6"/>
+<instance part="GND12" gate="1" x="157.48" y="190.5"/>
 <instance part="R16" gate="G$1" x="121.92" y="99.06" rot="R180"/>
 <instance part="NC7" gate="G$1" x="30.48" y="236.22" rot="MR0"/>
@@
 <instance part="IC2" gate="1" x="93.98" y="45.72"/>
 <instance part="P+11" gate="VCC" x="78.74" y="45.72" rot="MR270"/>
-<instance part="P+12" gate="1" x="111.76" y="45.72" rot="R270"/>
+<instance part="P+12" gate="1" x="109.22" y="45.72" rot="R270"/>
 <instance part="GND16" gate="1" x="93.98" y="25.4" rot="MR0"/>
 <instance part="JP2" gate="A" x="147.32" y="198.12"/>
 <instance part="JP3" gate="A" x="157.48" y="142.24"/>
-<instance part="D3" gate="1" x="93.98" y="53.34" rot="R180"/>
-<instance part="C2" gate="G$1" x="83.82" y="40.64"/>
-<instance part="C3" gate="G$1" x="104.14" y="40.64"/>
 </instances>
 <busses>
@@
 </segment>
 <segment>
+<pinref part="GND12" gate="1" pin="GND"/>
+<wire x1="160.02" y1="203.2" x2="157.48" y2="203.2" width="0.1524" layer="91"/>
+<wire x1="157.48" y1="203.2" x2="157.48" y2="200.66" width="0.1524" layer="91"/>
+<wire x1="157.48" y1="200.66" x2="157.48" y2="198.12" width="0.1524" layer="91"/>
+<wire x1="157.48" y1="198.12" x2="157.48" y2="195.58" width="0.1524" layer="91"/>
+<wire x1="157.48" y1="195.58" x2="157.48" y2="193.04" width="0.1524" layer="91"/>
+<wire x1="160.02" y1="200.66" x2="157.48" y2="200.66" width="0.1524" layer="91"/>
+<junction x="157.48" y="200.66"/>
+<wire x1="160.02" y1="198.12" x2="157.48" y2="198.12" width="0.1524" layer="91"/>
+<junction x="157.48" y="198.12"/>
+<wire x1="160.02" y1="195.58" x2="157.48" y2="195.58" width="0.1524" layer="91"/>
+<junction x="157.48" y="195.58"/>
+</segment>
+<segment>
 <pinref part="GND13" gate="1" pin="GND"/>
 <wire x1="154.94" y1="137.16" x2="147.32" y2="137.16" width="0.1524" layer="91"/>
@@
 <pinref part="GND16" gate="1" pin="GND"/>
 <pinref part="IC2" gate="1" pin="GND"/>
-<wire x1="93.98" y1="27.94" x2="93.98" y2="33.02" width="0.1524" layer="91"/>
-<pinref part="C2" gate="G$1" pin="2"/>
-<wire x1="93.98" y1="33.02" x2="93.98" y2="38.1" width="0.1524" layer="91"/>
-<wire x1="83.82" y1="35.56" x2="83.82" y2="33.02" width="0.1524" layer="91"/>
-<wire x1="83.82" y1="33.02" x2="93.98" y2="33.02" width="0.1524" layer="91"/>
-<junction x="93.98" y="33.02"/>
-<pinref part="C3" gate="G$1" pin="2"/>
-<wire x1="104.14" y1="35.56" x2="104.14" y2="33.02" width="0.1524" layer="91"/>
-<wire x1="104.14" y1="33.02" x2="93.98" y2="33.02" width="0.1524" layer="91"/>
+<wire x1="93.98" y1="27.94" x2="93.98" y2="38.1" width="0.1524" layer="91"/>
 </segment>
 </net>
@@
 <pinref part="P+12" gate="1" pin="+5V"/>
 <pinref part="IC2" gate="1" pin="OUT"/>
-<wire x1="109.22" y1="45.72" x2="104.14" y2="45.72" width="0.1524" layer="91"/>
-<pinref part="D3" gate="1" pin="A"/>
-<wire x1="104.14" y1="45.72" x2="101.6" y2="45.72" width="0.1524" layer="91"/>
-<wire x1="96.52" y1="53.34" x2="104.14" y2="53.34" width="0.1524" layer="91"/>
-<wire x1="104.14" y1="53.34" x2="104.14" y2="45.72" width="0.1524" layer="91"/>
-<junction x="104.14" y="45.72"/>
-<pinref part="C3" gate="G$1" pin="1"/>
-<wire x1="104.14" y1="43.18" x2="104.14" y2="45.72" width="0.1524" layer="91"/>
+<wire x1="106.68" y1="45.72" x2="101.6" y2="45.72" width="0.1524" layer="91"/>
 </segment>
 </net>
@@
 <pinref part="P+11" gate="VCC" pin="VCC"/>
 <pinref part="IC2" gate="1" pin="IN"/>
-<wire x1="81.28" y1="45.72" x2="83.82" y2="45.72" width="0.1524" layer="91"/>
-<pinref part="D3" gate="1" pin="C"/>
-<wire x1="83.82" y1="45.72" x2="86.36" y2="45.72" width="0.1524" layer="91"/>
-<wire x1="91.44" y1="53.34" x2="83.82" y2="53.34" width="0.1524" layer="91"/>
-<wire x1="83.82" y1="53.34" x2="83.82" y2="45.72" width="0.1524" layer="91"/>
-<junction x="83.82" y="45.72"/>
-<pinref part="C2" gate="G$1" pin="1"/>
-<wire x1="83.82" y1="43.18" x2="83.82" y2="45.72" width="0.1524" layer="91"/>
-</segment>
-</net>
+<wire x1="81.28" y1="45.72" x2="86.36" y2="45.72" width="0.1524" layer="91"/>
+</segment>
+</net>
